File: Production/Panel (2).brd (EAGLE design)
At the start: 138.4 x 138.4 mm, 205 parts, among them J1 DOUBLE_LED_PAD, J10 DOUBLE_LED_PAD, J11 DOUBLE_LED_PAD, J12 DOUBLE_LED_PAD, J2 DOUBLE_LED_PAD, J3 DOUBLE_LED_PAD, J4 DOUBLE_LED_PAD, J5 DOUBLE_LED_PAD, J6 DOUBLE_LED_PAD, J7 DOUBLE_LED_PAD, J8 DOUBLE_LED_PAD, J9 DOUBLE_LED_PAD

Commit message: Cleaning repo, changing name, pre review
Parts:
- removed E$2: (no value), SparkFun-Aesthetics:FIDUCIAL-MICRO
- removed FRAME3: FRAME-LETTER, SparkFun-Aesthetics:CREATIVE_COMMONS
- removed J10, J11, J12: DOUBLE_LED_PAD, Andy:DOUBLELEDPAD
- removed U$25: (no value), buzzard_labels (25):G4
- removed U$26: (no value), buzzard_labels (25):DO3
- removed U$27: (no value), buzzard_labels (25):CO1
- removed U$28: (no value), buzzard_labels (26):CI6
- removed U$29: (no value), buzzard_labels (26):DI4
- removed U$30: (no value), buzzard_labels (28):100_APA102_LED#S0
- U$11: device buzzard_labels (22):CHROMADOT5 -> buzzard_labels (28):100_APA102_LED#S0
- U$12: device buzzard_labels (25):5V6 -> buzzard_labels (25):DO3
- U$13, U$22: device buzzard_labels (25):5V6 -> buzzard_labels (25):CO1
- U$14: device buzzard_labels (25):G4 -> buzzard_labels (26):CI6
- U$15, U$24: device buzzard_labels (25):G4 -> buzzard_labels (26):DI4
- U$16: device buzzard_labels (25):DO3 -> buzzard_labels (28):40_APA102_LED#S1
- U$17: device buzzard_labels (25):CO1 -> buzzard_labels (22):CHROMADOT5
- U$18: device buzzard_labels (26):CI6 -> buzzard_labels (22):20_APA102_LED#S6
- U$19: device buzzard_labels (26):DI4 -> buzzard_labels (25):5V6
- U$2: device buzzard_labels (22):20_APA102_LED#S6 -> buzzard_labels (22):CHROMADOT5
- U$20: device buzzard_labels (28):40_APA102_LED#S1 -> buzzard_labels (25):G4
- U$21: device buzzard_labels (22):CHROMADOT5 -> buzzard_labels (25):DO3
- U$23: device buzzard_labels (25):5V6 -> buzzard_labels (26):CI6
- moved D68 121.2 mm to (32.3, 8.40), turned to 331.2 degrees
- moved D70 121.2 mm to (39.2, 5.15), turned to 338.4 degrees
- moved D63 121.2 mm to (17.3, 20.0), turned to 313.2 degrees
- moved D66 121.2 mm to (25.9, 12.5), turned to 324 degrees
- moved D64 121.2 mm to (20.0, 17.3), turned to 316.8 degrees
- moved D65 121.2 mm to (22.9, 14.8), turned to 320.4 degrees
- moved D69 121.2 mm to (35.7, 6.67), turned to 334.8 degrees
- moved D62 121.2 mm to (14.8, 22.9), turned to 309.6 degrees
- moved D67 121.2 mm to (29.1, 10.3), turned to 327.6 degrees
- moved D84 115.5 mm to (90.8, 8.40), turned to 28.8 degrees
- moved D61 115.5 mm to (12.5, 25.9), turned to 306 degrees
- moved D86 115.5 mm to (97.3, 12.5), turned to 36 degrees
- moved D91 115.5 mm to (110.7, 25.9), turned to 54 degrees
- moved D96 115.5 mm to (119.3, 42.8), turned to 72 degrees
- moved D98 115.5 mm to (121.2, 50.2), turned to 79.2 degrees
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Connections:
- removed net 5V: D1.VDD, D1.VDDPAD, D10.VDD, D10.VDDPAD, D11.VDD, D11.VDDPAD, D12.VDD, D12.VDDPAD, D13.VDD, D13.VDDPAD, D14.VDD, D14.VDDPAD, D15.VDD, D15.VDDPAD, D16.VDD, D16.VDDPAD, D17.VDD, D17.VDDPAD, D18.VDD, D18.VDDPAD, D19.VDD, D19.VDDPAD, D2.VDD, D2.VDDPAD, D20.VDD, D20.VDDPAD, D3.VDD, D3.VDDPAD, D4.VDD, D4.VDDPAD, D5.VDD, D5.VDDPAD, D6.VDD, D6.VDDPAD, D7.VDD, D7.VDDPAD, D8.VDD, D8.VDDPAD, D9.VDD, D9.VDDPAD, J1.P$2, J3.P$2
- removed net GND: D1.GND, D1.GNDPAD, D10.GND, D10.GNDPAD, D11.GND, D11.GNDPAD, D12.GND, D12.GNDPAD, D13.GND, D13.GNDPAD, D14.GND, D14.GNDPAD, D15.GND, D15.GNDPAD, D16.GND, D16.GNDPAD, D17.GND, D17.GNDPAD, D18.GND, D18.GNDPAD, D19.GND, D19.GNDPAD, D2.GND, D2.GNDPAD, D20.GND, D20.GNDPAD, D3.GND, D3.GNDPAD, D4.GND, D4.GNDPAD, D5.GND, D5.GNDPAD, D6.GND, D6.GNDPAD, D7.GND, D7.GNDPAD, D8.GND, D8.GNDPAD, D9.GND, D9.GNDPAD, J1.P$1, J3.P$1
- removed net N$126 (its old number): D61.SDO, D71.SDI
- removed net N$133 (its old number): D60.CKO, J7.P$2
- removed net N$134 (its old number): D60.SDO, J7.P$1
- removed net N$142 (its old number): D62.SDI, D78.SDO
- removed net N$160 (its old number): D70.CKO, D79.CKI
- removed net N$233 (its old number): D118.SDO, D119.SDI
- removed net N$236 (its old number): D118.CKO, D119.CKI
- removed net N$281 (its old number): D100.CKO, D101.CKI
- removed net N$282 (its old number): D100.SDO, D101.SDI
- removed net N$301 (its old number): D150.CKO, D151.CKI
- removed net N$302 (its old number): D150.SDO, D151.SDI
- removed net N$315 (its old number): D158.SDO, D159.SDI
- removed net N$318 (its old number): D158.CKO, D159.CKI
- removed net N$323 (its old number): D160.SDO, J12.P$1
- removed net N$43 (its old number): D21.CKI, J6.P$2
- removed net N$46 (its old number): D21.SDO, D31.SDI
- removed net N$59 (its old number): D22.CKI, D38.CKO
- removed net N$75 (its old number): D30.SDO, D39.SDI
- removed net N$78 (its old number): D30.CKO, D39.CKI
- new net 5V3: D1.VDD, D1.VDDPAD, D10.VDD, D10.VDDPAD, D100.VDD, D100.VDDPAD, D11.VDD, D11.VDDPAD, D12.VDD, D12.VDDPAD, D13.VDD, D13.VDDPAD, D14.VDD, D14.VDDPAD, D15.VDD, D15.VDDPAD, D16.VDD, D16.VDDPAD, D17.VDD, D17.VDDPAD, D18.VDD, D18.VDDPAD, D19.VDD, D19.VDDPAD, D2.VDD, D2.VDDPAD, D20.VDD, D20.VDDPAD, D21.VDD, D21.VDDPAD, D22.VDD, D22.VDDPAD, D23.VDD, D23.VDDPAD, D24.VDD, D24.VDDPAD, D25.VDD, D25.VDDPAD, D26.VDD, D26.VDDPAD, D27.VDD, D27.VDDPAD, D28.VDD, D28.VDDPAD, D29.VDD, D29.VDDPAD, D3.VDD, D3.VDDPAD, D30.VDD, D30.VDDPAD, D31.VDD, D31.VDDPAD, D32.VDD, D32.VDDPAD, D33.VDD, D33.VDDPAD, D34.VDD, D34.VDDPAD, D35.VDD, D35.VDDPAD, D36.VDD, D36.VDDPAD, D37.VDD, D37.VDDPAD, D38.VDD, D38.VDDPAD, D39.VDD, D39.VDDPAD, D4.VDD, D4.VDDPAD, D40.VDD, D40.VDDPAD, D41.VDD, D41.VDDPAD, D42.VDD, D42.VDDPAD, D43.VDD, D43.VDDPAD, D44.VDD, D44.VDDPAD, D45.VDD, D45.VDDPAD, D46.VDD, D46.VDDPAD, D47.VDD, D47.VDDPAD, D48.VDD, D48.VDDPAD, D49.VDD, D49.VDDPAD, D5.VDD, D5.VDDPAD, D50.VDD, D50.VDDPAD, D51.VDD, D51.VDDPAD, D52.VDD, D52.VDDPAD, D53.VDD, D53.VDDPAD, D54.VDD, D54.VDDPAD, D55.VDD, D55.VDDPAD, D56.VDD, D56.VDDPAD, D57.VDD, D57.VDDPAD, D58.VDD, D58.VDDPAD, D59.VDD, D59.VDDPAD, D6.VDD, D6.VDDPAD, D60.VDD, D60.VDDPAD, D61.VDD, D61.VDDPAD, D62.VDD, D62.VDDPAD, D63.VDD, D63.VDDPAD, D64.VDD, D64.VDDPAD, D65.VDD, D65.VDDPAD, D66.VDD, D66.VDDPAD, D67.VDD, D67.VDDPAD, D68.VDD, D68.VDDPAD, D69.VDD, D69.VDDPAD, D7.VDD, D7.VDDPAD, D70.VDD, D70.VDDPAD, D71.VDD, D71.VDDPAD, D72.VDD, D72.VDDPAD, D73.VDD, D73.VDDPAD, D74.VDD, D74.VDDPAD, D75.VDD, D75.VDDPAD, D76.VDD, D76.VDDPAD, D77.VDD, D77.VDDPAD, D78.VDD, D78.VDDPAD, D79.VDD, D79.VDDPAD, D8.VDD, D8.VDDPAD, D80.VDD, D80.VDDPAD, D81.VDD, D81.VDDPAD, D82.VDD, D82.VDDPAD, D83.VDD, D83.VDDPAD, D84.VDD, D84.VDDPAD, D85.VDD, D85.VDDPAD, D86.VDD, D86.VDDPAD, D87.VDD, D87.VDDPAD, D88.VDD, D88.VDDPAD, D89.VDD, D89.VDDPAD, D9.VDD, D9.VDDPAD, D90.VDD, D90.VDDPAD, D91.VDD, D91.VDDPAD, D92.VDD, D92.VDDPAD, D93.VDD, D93.VDDPAD, D94.VDD, D94.VDDPAD, D95.VDD, D95.VDDPAD, D96.VDD, D96.VDDPAD, D97.VDD, D97.VDDPAD, D98.VDD, D98.VDDPAD, D99.VDD, D99.VDDPAD, J1.P$2
- new net GND3: D1.GND, D1.GNDPAD, D10.GND, D10.GNDPAD, D100.GND, D100.GNDPAD, D11.GND, D11.GNDPAD, D12.GND, D12.GNDPAD, D13.GND, D13.GNDPAD, D14.GND, D14.GNDPAD, D15.GND, D15.GNDPAD, D16.GND, D16.GNDPAD, D17.GND, D17.GNDPAD, D18.GND, D18.GNDPAD, D19.GND, D19.GNDPAD, D2.GND, D2.GNDPAD, D20.GND, D20.GNDPAD, D21.GND, D21.GNDPAD, D22.GND, D22.GNDPAD, D23.GND, D23.GNDPAD, D24.GND, D24.GNDPAD, D25.GND, D25.GNDPAD, D26.GND, D26.GNDPAD, D27.GND, D27.GNDPAD, D28.GND, D28.GNDPAD, D29.GND, D29.GNDPAD, D3.GND, D3.GNDPAD, D30.GND, D30.GNDPAD, D31.GND, D31.GNDPAD, D32.GND, D32.GNDPAD, D33.GND, D33.GNDPAD, D34.GND, D34.GNDPAD, D35.GND, D35.GNDPAD, D36.GND, D36.GNDPAD, D37.GND, D37.GNDPAD, D38.GND, D38.GNDPAD, D39.GND, D39.GNDPAD, D4.GND, D4.GNDPAD, D40.GND, D40.GNDPAD, D41.GND, D41.GNDPAD, D42.GND, D42.GNDPAD, D43.GND, D43.GNDPAD, D44.GND, D44.GNDPAD, D45.GND, D45.GNDPAD, D46.GND, D46.GNDPAD, D47.GND, D47.GNDPAD, D48.GND, D48.GNDPAD, D49.GND, D49.GNDPAD, D5.GND, D5.GNDPAD, D50.GND, D50.GNDPAD, D51.GND, D51.GNDPAD, D52.GND, D52.GNDPAD, D53.GND, D53.GNDPAD, D54.GND, D54.GNDPAD, D55.GND, D55.GNDPAD, D56.GND, D56.GNDPAD, D57.GND, D57.GNDPAD, D58.GND, D58.GNDPAD, D59.GND, D59.GNDPAD, D6.GND, D6.GNDPAD, D60.GND, D60.GNDPAD, D61.GND, D61.GNDPAD, D62.GND, D62.GNDPAD, D63.GND, D63.GNDPAD, D64.GND, D64.GNDPAD, D65.GND, D65.GNDPAD, D66.GND, D66.GNDPAD, D67.GND, D67.GNDPAD, D68.GND, D68.GNDPAD, D69.GND, D69.GNDPAD, D7.GND, D7.GNDPAD, D70.GND, D70.GNDPAD, D71.GND, D71.GNDPAD, D72.GND, D72.GNDPAD, D73.GND, D73.GNDPAD, D74.GND, D74.GNDPAD, D75.GND, D75.GNDPAD, D76.GND, D76.GNDPAD, D77.GND, D77.GNDPAD, D78.GND, D78.GNDPAD, D79.GND, D79.GNDPAD, D8.GND, D8.GNDPAD, D80.GND, D80.GNDPAD, D81.GND, D81.GNDPAD, D82.GND, D82.GNDPAD, D83.GND, D83.GNDPAD, D84.GND, D84.GNDPAD, D85.GND, D85.GNDPAD, D86.GND, D86.GNDPAD, D87.GND, D87.GNDPAD, D88.GND, D88.GNDPAD, D89.GND, D89.GNDPAD, D9.GND, D9.GNDPAD, D90.GND, D90.GNDPAD, D91.GND, D91.GNDPAD, D92.GND, D92.GNDPAD, D93.GND, D93.GNDPAD, D94.GND, D94.GNDPAD, D95.GND, D95.GNDPAD, D96.GND, D96.GNDPAD, D97.GND, D97.GNDPAD, D98.GND, D98.GNDPAD, D99.GND, D99.GNDPAD, J1.P$1
- new net N$122: D60.CKO, D61.CKI
- new net N$140: D70.CKO, D71.CKI
- new net N$154: D78.SDO, D79.SDI
- new net N$162: D100.SDO, J3.P$1
- new net N$163: D100.CKO, J3.P$2
- new net N$205: D101.CKO, D111.CKI
- new net N$206: D101.SDO, D111.SDI
- new net N$235: D110.SDO, D119.SDI
- new net N$238: D110.CKO, D119.CKI
- new net N$283: D140.CKO, J6.P$2
- new net N$284: D140.SDO, J6.P$1
- new net N$287: D141.CKO, D151.CKI
- new net N$288: D141.SDO, D151.SDI
- new net N$303: D142.CKI, D158.CKO
- new net N$304: D142.SDI, D158.SDO
- new net N$321: D150.SDO, D159.SDI
- new net N$61: D30.SDO, D31.SDI
- new net N$74: D38.SDO, D39.SDI
- new net N$77: D38.CKO, D39.CKI
- net 5V1: now also D101.VDD, D101.VDDPAD, D102.VDD, D102.VDDPAD, D103.VDD, D103.VDDPAD, D104.VDD, D104.VDDPAD, D105.VDD, D105.VDDPAD, D106.VDD, D106.VDDPAD, D107.VDD, D107.VDDPAD, D108.VDD, D108.VDDPAD, D109.VDD, D109.VDDPAD, D110.VDD, D110.VDDPAD, D111.VDD, D111.VDDPAD, D112.VDD, D112.VDDPAD, D113.VDD, D113.VDDPAD, D114.VDD, D114.VDDPAD, D115.VDD, D115.VDDPAD, D116.VDD, D116.VDDPAD, D117.VDD, D117.VDDPAD, D118.VDD, D118.VDDPAD, D119.VDD, D119.VDDPAD, D120.VDD, D120.VDDPAD, D121.VDD, D121.VDDPAD, D122.VDD, D122.VDDPAD, D123.VDD, D123.VDDPAD, D124.VDD, D124.VDDPAD, D125.VDD, D125.VDDPAD, D126.VDD, D126.VDDPAD, D127.VDD, D127.VDDPAD, D128.VDD, D128.VDDPAD, D129.VDD, D129.VDDPAD, D130.VDD, D130.VDDPAD, D131.VDD, D131.VDDPAD, D132.VDD, D132.VDDPAD, D133.VDD, D133.VDDPAD, D134.VDD, D134.VDDPAD, D135.VDD, D135.VDDPAD, D136.VDD, D136.VDDPAD, D137.VDD, D137.VDDPAD, D138.VDD, D138.VDDPAD, D139.VDD, D139.VDDPAD, D140.VDD, D140.VDDPAD, J4.P$2; no longer D21.VDD, D21.VDDPAD, D22.VDD, D22.VDDPAD, D23.VDD, D23.VDDPAD, D24.VDD, D24.VDDPAD, D25.VDD, D25.VDDPAD, D26.VDD, D26.VDDPAD, D27.VDD, D27.VDDPAD, D28.VDD, D28.VDDPAD, D29.VDD, D29.VDDPAD, D30.VDD, D30.VDDPAD, D31.VDD, D31.VDDPAD, D32.VDD, D32.VDDPAD, D33.VDD, D33.VDDPAD, D34.VDD, D34.VDDPAD, D35.VDD, D35.VDDPAD, D36.VDD, D36.VDDPAD, D37.VDD, D37.VDDPAD, D38.VDD, D38.VDDPAD, D39.VDD, D39.VDDPAD, D40.VDD, D40.VDDPAD, D41.VDD, D41.VDDPAD, D42.VDD, D42.VDDPAD, D43.VDD, D43.VDDPAD, D44.VDD, D44.VDDPAD, D45.VDD, D45.VDDPAD, D46.VDD, D46.VDDPAD, D47.VDD, D47.VDDPAD, D48.VDD, D48.VDDPAD, D49.VDD, D49.VDDPAD, D50.VDD, D50.VDDPAD, D51.VDD, D51.VDDPAD, D52.VDD, D52.VDDPAD, D53.VDD, D53.VDDPAD, D54.VDD, D54.VDDPAD, D55.VDD, D55.VDDPAD, D56.VDD, D56.VDDPAD, D57.VDD, D57.VDDPAD, D58.VDD, D58.VDDPAD, D59.VDD, D59.VDDPAD, D60.VDD, D60.VDDPAD, J5.P$2, J8.P$2
- net 5V2: now also J7.P$2; no longer D100.VDD, D100.VDDPAD, D101.VDD, D101.VDDPAD, D102.VDD, D102.VDDPAD, D103.VDD, D103.VDDPAD, D104.VDD, D104.VDDPAD, D105.VDD, D105.VDDPAD, D106.VDD, D106.VDDPAD, D107.VDD, D107.VDDPAD, D108.VDD, D108.VDDPAD, D109.VDD, D109.VDDPAD, D110.VDD, D110.VDDPAD, D111.VDD, D111.VDDPAD, D112.VDD, D112.VDDPAD, D113.VDD, D113.VDDPAD, D114.VDD, D114.VDDPAD, D115.VDD, D115.VDDPAD, D116.VDD, D116.VDDPAD, D117.VDD, D117.VDDPAD, D118.VDD, D118.VDDPAD, D119.VDD, D119.VDDPAD, D120.VDD, D120.VDDPAD, D121.VDD, D121.VDDPAD, D122.VDD, D122.VDDPAD, D123.VDD, D123.VDDPAD, D124.VDD, D124.VDDPAD, D125.VDD, D125.VDDPAD, D126.VDD, D126.VDDPAD, D127.VDD, D127.VDDPAD, D128.VDD, D128.VDDPAD, D129.VDD, D129.VDDPAD, D130.VDD, D130.VDDPAD, D131.VDD, D131.VDDPAD, D132.VDD, D132.VDDPAD, D133.VDD, D133.VDDPAD, D134.VDD, D134.VDDPAD, D135.VDD, D135.VDDPAD, D136.VDD, D136.VDDPAD, D137.VDD, D137.VDDPAD, D138.VDD, D138.VDDPAD, D139.VDD, D139.VDDPAD, D140.VDD, D140.VDDPAD, D61.VDD, D61.VDDPAD, D62.VDD, D62.VDDPAD, D63.VDD, D63.VDDPAD, D64.VDD, D64.VDDPAD, D65.VDD, D65.VDDPAD, D66.VDD, D66.VDDPAD, D67.VDD, D67.VDDPAD, D68.VDD, D68.VDDPAD, D69.VDD, D69.VDDPAD, D70.VDD, D70.VDDPAD, D71.VDD, D71.VDDPAD, D72.VDD, D72.VDDPAD, D73.VDD, D73.VDDPAD, D74.VDD, D74.VDDPAD, D75.VDD, D75.VDDPAD, D76.VDD, D76.VDDPAD, D77.VDD, D77.VDDPAD, D78.VDD, D78.VDDPAD, D79.VDD, D79.VDDPAD, D80.VDD, D80.VDDPAD, D81.VDD, D81.VDDPAD, D82.VDD, D82.VDDPAD, D83.VDD, D83.VDDPAD, D84.VDD, D84.VDDPAD, D85.VDD, D85.VDDPAD, D86.VDD, D86.VDDPAD, D87.VDD, D87.VDDPAD, D88.VDD, D88.VDDPAD, D89.VDD, D89.VDDPAD, D90.VDD, D90.VDDPAD, D91.VDD, D91.VDDPAD, D92.VDD, D92.VDDPAD, D93.VDD, D93.VDDPAD, D94.VDD, D94.VDDPAD, D95.VDD, D95.VDDPAD, D96.VDD, D96.VDDPAD, D97.VDD, D97.VDDPAD, D98.VDD, D98.VDDPAD, D99.VDD, D99.VDDPAD, J11.P$2, J9.P$2
- net GND1: now also D101.GND, D101.GNDPAD, D102.GND, D102.GNDPAD, D103.GND, D103.GNDPAD, D104.GND, D104.GNDPAD, D105.GND, D105.GNDPAD, D106.GND, D106.GNDPAD, D107.GND, D107.GNDPAD, D108.GND, D108.GNDPAD, D109.GND, D109.GNDPAD, D110.GND, D110.GNDPAD, D111.GND, D111.GNDPAD, D112.GND, D112.GNDPAD, D113.GND, D113.GNDPAD, D114.GND, D114.GNDPAD, D115.GND, D115.GNDPAD, D116.GND, D116.GNDPAD, D117.GND, D117.GNDPAD, D118.GND, D118.GNDPAD, D119.GND, D119.GNDPAD, D120.GND, D120.GNDPAD, D121.GND, D121.GNDPAD, D122.GND, D122.GNDPAD, D123.GND, D123.GNDPAD, D124.GND, D124.GNDPAD, D125.GND, D125.GNDPAD, D126.GND, D126.GNDPAD, D127.GND, D127.GNDPAD, D128.GND, D128.GNDPAD, D129.GND, D129.GNDPAD, D130.GND, D130.GNDPAD, D131.GND, D131.GNDPAD, D132.GND, D132.GNDPAD, D133.GND, D133.GNDPAD, D134.GND, D134.GNDPAD, D135.GND, D135.GNDPAD, D136.GND, D136.GNDPAD, D137.GND, D137.GNDPAD, D138.GND, D138.GNDPAD, D139.GND, D139.GNDPAD, D140.GND, D140.GNDPAD, J4.P$1; no longer D21.GND, D21.GNDPAD, D22.GND, D22.GNDPAD, D23.GND, D23.GNDPAD, D24.GND, D24.GNDPAD, D25.GND, D25.GNDPAD, D26.GND, D26.GNDPAD, D27.GND, D27.GNDPAD, D28.GND, D28.GNDPAD, D29.GND, D29.GNDPAD, D30.GND, D30.GNDPAD, D31.GND, D31.GNDPAD, D32.GND, D32.GNDPAD, D33.GND, D33.GNDPAD, D34.GND, D34.GNDPAD, D35.GND, D35.GNDPAD, D36.GND, D36.GNDPAD, D37.GND, D37.GNDPAD, D38.GND, D38.GNDPAD, D39.GND, D39.GNDPAD, D40.GND, D40.GNDPAD, D41.GND, D41.GNDPAD, D42.GND, D42.GNDPAD, D43.GND, D43.GNDPAD, D44.GND, D44.GNDPAD, D45.GND, D45.GNDPAD, D46.GND, D46.GNDPAD, D47.GND, D47.GNDPAD, D48.GND, D48.GNDPAD, D49.GND, D49.GNDPAD, D50.GND, D50.GNDPAD, D51.GND, D51.GNDPAD, D52.GND, D52.GNDPAD, D53.GND, D53.GNDPAD, D54.GND, D54.GNDPAD, D55.GND, D55.GNDPAD, D56.GND, D56.GNDPAD, D57.GND, D57.GNDPAD, D58.GND, D58.GNDPAD, D59.GND, D59.GNDPAD, D60.GND, D60.GNDPAD, J5.P$1, J8.P$1
- net GND2: now also J7.P$1; no longer D100.GND, D100.GNDPAD, D101.GND, D101.GNDPAD, D102.GND, D102.GNDPAD, D103.GND, D103.GNDPAD, D104.GND, D104.GNDPAD, D105.GND, D105.GNDPAD, D106.GND, D106.GNDPAD, D107.GND, D107.GNDPAD, D108.GND, D108.GNDPAD, D109.GND, D109.GNDPAD, D110.GND, D110.GNDPAD, D111.GND, D111.GNDPAD, D112.GND, D112.GNDPAD, D113.GND, D113.GNDPAD, D114.GND, D114.GNDPAD, D115.GND, D115.GNDPAD, D116.GND, D116.GNDPAD, D117.GND, D117.GNDPAD, D118.GND, D118.GNDPAD, D119.GND, D119.GNDPAD, D120.GND, D120.GNDPAD, D121.GND, D121.GNDPAD, D122.GND, D122.GNDPAD, D123.GND, D123.GNDPAD, D124.GND, D124.GNDPAD, D125.GND, D125.GNDPAD, D126.GND, D126.GNDPAD, D127.GND, D127.GNDPAD, D128.GND, D128.GNDPAD, D129.GND, D129.GNDPAD, D130.GND, D130.GNDPAD, D131.GND, D131.GNDPAD, D132.GND, D132.GNDPAD, D133.GND, D133.GNDPAD, D134.GND, D134.GNDPAD, D135.GND, D135.GNDPAD, D136.GND, D136.GNDPAD, D137.GND, D137.GNDPAD, D138.GND, D138.GNDPAD, D139.GND, D139.GNDPAD, D140.GND, D140.GNDPAD, D61.GND, D61.GNDPAD, D62.GND, D62.GNDPAD, D63.GND, D63.GNDPAD, D64.GND, D64.GNDPAD, D65.GND, D65.GNDPAD, D66.GND, D66.GNDPAD, D67.GND, D67.GNDPAD, D68.GND, D68.GNDPAD, D69.GND, D69.GNDPAD, D70.GND, D70.GNDPAD, D71.GND, D71.GNDPAD, D72.GND, D72.GNDPAD, D73.GND, D73.GNDPAD, D74.GND, D74.GNDPAD, D75.GND, D75.GNDPAD, D76.GND, D76.GNDPAD, D77.GND, D77.GNDPAD, D78.GND, D78.GNDPAD, D79.GND, D79.GNDPAD, D80.GND, D80.GNDPAD, D81.GND, D81.GNDPAD, D82.GND, D82.GNDPAD, D83.GND, D83.GNDPAD, D84.GND, D84.GNDPAD, D85.GND, D85.GNDPAD, D86.GND, D86.GNDPAD, D87.GND, D87.GNDPAD, D88.GND, D88.GNDPAD, D89.GND, D89.GNDPAD, D90.GND, D90.GNDPAD, D91.GND, D91.GNDPAD, D92.GND, D92.GNDPAD, D93.GND, D93.GNDPAD, D94.GND, D94.GNDPAD, D95.GND, D95.GNDPAD, D96.GND, D96.GNDPAD, D97.GND, D97.GNDPAD, D98.GND, D98.GNDPAD, D99.GND, D99.GNDPAD, J11.P$1, J9.P$1
- net N$123: now also D60.SDO, D61.SDI; no longer D61.CKI, J10.P$2
- net N$124: now also D61.CKO, D62.CKI; no longer D61.SDI, J10.P$1
- net N$125: now also D61.SDO, D62.SDI; no longer D61.CKO, D71.CKI
- net N$141: now also D70.SDO, D71.SDI; no longer D62.CKI, D78.CKO
- net N$157: now also D78.CKO, D79.CKI; no longer D70.SDO, D79.SDI
- net N$203: now also D101.CKI, J5.P$2; no longer D101.CKO, D102.CKI
- net N$204: now also D101.SDI, J5.P$1; no longer D101.SDO, D102.SDI
- net N$219: now also D102.CKI, D118.CKO; no longer D110.CKO, D111.CKI
- net N$220: now also D102.SDI, D118.SDO; no longer D110.SDO, D111.SDI
- net N$285: now also D141.CKI, J8.P$2; no longer D141.CKO, D142.CKI
- net N$286: now also D141.SDI, J8.P$1; no longer D141.SDO, D142.SDI
- net N$324: now also D150.CKO, D159.CKI; no longer D160.CKO, J12.P$2
- net N$325: now also D160.CKO, J9.P$2; no longer D140.CKO, D141.CKI
- net N$326: now also D160.SDO, J9.P$1; no longer D140.SDO, D141.SDI
- net N$41: now also D21.CKI; no longer J4.P$2
- net N$42: now also D21.SDI; no longer J4.P$1
- net N$44: now also D21.CKO, D22.CKI; no longer D21.SDI, J6.P$1
- net N$45: now also D21.SDO, D22.SDI; no longer D21.CKO, D31.CKI
- net N$60: now also D30.CKO, D31.CKI; no longer D22.SDI, D38.SDO
Routing:
- net 5V3: track 0.00 -> 230.1 mm, vias 0 -> 101
- net 5V2: track 231.0 -> 37.6 mm, vias 101 -> 20
- net 5V: track 38.0 -> 0.00 mm, vias 20 -> 0
- net GND: track 5.96 -> 0.00 mm, vias 3 -> 0
- net N$323 (its old number): track 4.86 -> 0.00 mm, vias 1 -> 0
- net GND1: track 12.3 -> 7.43 mm, vias 5 -> 4
- net 5V1: track 85.9 -> 81.1 mm
- net N$163: track 0.00 -> 4.63 mm, vias 0 -> 1
- net N$134 (its old number): track 4.55 -> 0.00 mm, vias 1 -> 0
- net N$162: track 0.00 -> 4.00 mm, vias 0 -> 1
- net N$284: track 0.00 -> 3.85 mm, vias 0 -> 1
- net GND3: track 0.00 -> 3.59 mm, vias 0 -> 2
- net N$43 (its old number): track 3.25 -> 0.00 mm, vias 1 -> 0
- net N$124: track 5.32 -> 2.11 mm, vias 1 -> 0
- net N$44: track 4.81 -> 2.12 mm, vias 1 -> 0
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- added copper zone on layer 16, net 5V3
- added copper zone on layer 1, net GND3
Other:
- board text added: "ROUTE OUT"
- board text added: "v03"
- board text removed: "v01"
